File: PCB/IR/03/IRRx.brd (EAGLE design)
At the start: 64 x 64 mm, 19 parts

Commit message: updated IRRx
Routing:
- net N$3: track 52.5 -> 48.0 mm
- net N$6: track 56.0 -> 54.7 mm
Other:
- board text added: "2019-11-02"
- board text added: "SWARMESH IRRx v3"
- board text removed: "SWARMESH IR v2 2019-09-16"
Changed lines of the file:
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@@
 <setting verticaltext="up"/>
 </settings>
-<grid distance="25" unitdist="mil" unit="mm" style="lines" multiple="1" display="no" altdistance="5" altunitdist="mil" altunit="mil"/>
+<grid distance="25" unitdist="mil" unit="mil" style="lines" multiple="1" display="no" altdistance="5" altunitdist="mil" altunit="mil"/>
 <layers>
 <layer number="1" name="Top" color="4" fill="1" visible="yes" active="yes"/>
@@
 <plain>
 <circle x="30" y="32" radius="32" width="0.1524" layer="20"/>
-<text x="-7.6708" y="35.433" size="1.778" layer="1">+</text>
-<text x="5.715" y="56.8452" size="1.778" layer="1" rot="R90">-</text>
-<text x="63.9826" y="53.975" size="1.143" layer="1" font="vector" rot="R135">SWARMESH
-IR v2
-2019-09-16</text>
+<text x="13.9192" y="13.843" size="1.778" layer="16" rot="MR0">+</text>
+<text x="12.065" y="8.5852" size="1.778" layer="16" rot="MR90">-</text>
+<text x="51.9176" y="45.085" size="1.778" layer="16" font="vector" ratio="15" rot="MR45">SWARMESH
+IRRx v3</text>
 <circle x="30" y="32" radius="9.398" width="0.1524" layer="20"/>
+<text x="36.6776" y="58.42" size="1.778" layer="16" font="vector" ratio="15" rot="MR0">2019-11-02</text>
 </plain>
 <attributes>
@@
 <contactref element="LED10" pad="K"/>
 <contactref element="R2" pad="2"/>
-<wire x1="15.08125" y1="23.495" x2="15.08125" y2="25.24125" width="0.5" layer="16"/>
-<wire x1="18.89125" y1="19.685" x2="15.08125" y2="23.495" width="0.5" layer="16"/>
 <wire x1="15.08125" y1="25.24125" x2="15.08" y2="25.27" width="0.5" layer="16"/>
-<wire x1="18.89125" y1="19.685" x2="18.923" y2="19.6088" width="0.5" layer="16"/>
 <wire x1="41.75125" y1="11.1125" x2="33.02" y2="11.1125" width="0.5" layer="16"/>
 <wire x1="22.86" y1="15.875" x2="19.05" y2="19.685" width="0.5" layer="16"/>
@@
 <wire x1="33.02" y1="11.1125" x2="27.6225" y2="11.1125" width="0.508" layer="16"/>
 <wire x1="27.6225" y1="11.1125" x2="22.86" y2="15.875" width="0.508" layer="16"/>
+<wire x1="18.923" y1="19.6088" x2="18.923" y2="21.3995" width="0.508" layer="16"/>
+<wire x1="18.923" y1="21.3995" x2="15.08125" y2="25.24125" width="0.508" layer="16"/>
 </signal>
 <signal name="N$2">
@@
 <contactref element="LED13" pad="K"/>
 <wire x1="15.875" y1="37.62375" x2="15.73" y2="37.635" width="0.5" layer="16"/>
-<wire x1="39.6875" y1="16.35125" x2="37.1475" y2="16.35125" width="0.5" layer="16"/>
 <wire x1="37.1475" y1="16.35125" x2="29.21" y2="16.35125" width="0.5" layer="16"/>
-<wire x1="39.6875" y1="16.35125" x2="40.62495" y2="15.4138" width="0.5" layer="16"/>
-<wire x1="40.62495" y1="15.4138" x2="41.275" y2="15.4138" width="0.5" layer="16"/>
 <wire x1="13.7668" y1="32.004" x2="13.7668" y2="35.51555" width="0.508" layer="16"/>
 <wire x1="13.7668" y1="35.51555" x2="15.875" y2="37.62375" width="0.508" layer="16"/>
@@
 <wire x1="18.7325" y1="44.1325" x2="18.57375" y2="43.97375" width="0.5" layer="16"/>
 <wire x1="18.7325" y1="44.1325" x2="18.8976" y2="44.323" width="0.5" layer="16"/>
-<wire x1="32.385" y1="17.30375" x2="27.78125" y2="17.30375" width="0.508" layer="16"/>
-<wire x1="27.78125" y1="17.30375" x2="19.685" y2="25.4" width="0.508" layer="16"/>
+<wire x1="32.385" y1="17.30375" x2="27.14625" y2="17.30375" width="0.508" layer="16"/>
+<wire x1="27.14625" y1="17.30375" x2="19.685" y2="24.765" width="0.508" layer="16"/>
 <wire x1="19.685" y1="27.06395" x2="16.51" y2="30.23895" width="0.508" layer="16"/>
 <wire x1="18.57375" y1="38.5030875" x2="18.57375" y2="39.37" width="0.508" layer="16"/>
 <wire x1="16.51" y1="36.4393375" x2="18.57375" y2="38.5030875" width="0.508" layer="16"/>
-<wire x1="19.685" y1="25.4" x2="19.685" y2="27.06395" width="0.508" layer="16"/>
+<wire x1="19.685" y1="24.765" x2="19.685" y2="27.06395" width="0.508" layer="16"/>
 <wire x1="16.51" y1="30.23895" x2="16.51" y2="36.4393375" width="0.508" layer="16"/>
 <wire x1="36.195" y1="17.30375" x2="40.13118125" y2="17.30375" width="0.508" layer="16"/>
@@
 <contactref element="JMUX" pad="4"/>
 <contactref element="LED14" pad="K"/>
-<wire x1="34.13125" y1="46.51375" x2="34.13125" y2="45.56125" width="0.5" layer="16"/>
-<wire x1="31.27375" y1="49.37125" x2="34.13125" y2="46.51375" width="0.5" layer="16"/>
-<wire x1="34.13125" y1="45.56125" x2="34.215" y2="45.4348" width="0.5" layer="16"/>
-<wire x1="31.27375" y1="49.37125" x2="31.2674" y2="49.5046" width="0.5" layer="16"/>
-<wire x1="40.48125" y1="18.0975" x2="45.085" y2="18.0975" width="0.5" layer="16"/>
+<wire x1="34.215" y1="45.4348" x2="32.0352" y2="45.4348" width="0.5" layer="16"/>
+<wire x1="32.0352" y1="45.4348" x2="31.4325" y2="46.0375" width="0.5" layer="16"/>
+<wire x1="31.4325" y1="46.0375" x2="31.2674" y2="49.5046" width="0.5" layer="16"/>
 <wire x1="39.6875" y1="18.89125" x2="40.48125" y2="18.0975" width="0.5" layer="16"/>
 <wire x1="39.6875" y1="22.86" x2="39.6875" y2="22.225" width="0.5" layer="16"/>
@@
 <wire x1="41.43375" y1="27.46375" x2="41.43375" y2="36.83" width="0.508" layer="16"/>
 <wire x1="39.6875" y1="25.7175" x2="41.43375" y2="27.46375" width="0.508" layer="16"/>
-<wire x1="45.085" y1="18.415" x2="45.72" y2="19.05" width="0.508" layer="16"/>
-<wire x1="45.085" y1="18.1015" x2="45.085" y2="18.415" width="0.508" layer="16"/>
-<wire x1="43.815" y1="18.1015" x2="45.085" y2="18.1015" width="0.508" layer="16"/>
-<wire x1="43.815" y1="18.2118" x2="43.815" y2="18.1015" width="0.508" layer="16"/>
-<wire x1="45.72" y1="19.05" x2="46.355" y2="19.685" width="0.508" layer="16"/>
-<wire x1="46.99" y1="19.685" x2="46.355" y2="19.685" width="0.508" layer="16"/>
-<wire x1="46.99" y1="19.685" x2="47.52815" y2="19.685" width="0.508" layer="16"/>
+<wire x1="46.355" y1="19.685" x2="47.52815" y2="19.685" width="0.508" layer="16"/>
 <wire x1="47.52815" y1="19.685" x2="49.019075" y2="18.194075" width="0.508" layer="16"/>
-<wire x1="45.085" y1="18.0975" x2="43.815" y2="18.2118" width="0" layer="19" extent="16-16"/>
+<wire x1="40.48125" y1="18.0975" x2="44.7675" y2="18.0975" width="0.508" layer="16"/>
+<wire x1="44.7675" y1="18.0975" x2="46.355" y2="19.685" width="0.508" layer="16"/>
 </signal>
 <signal name="N$6">
@@
 <wire x1="43.18" y1="47.625" x2="43.65625" y2="47.14875" width="0.508" layer="16"/>
 <wire x1="43.65625" y1="47.14875" x2="43.65625" y2="44.1325" width="0.508" layer="16"/>
-<wire x1="43.6372" y1="44.3738" x2="47.0662" y2="44.3738" width="0.508" layer="16"/>
-<wire x1="53.34" y1="38.1" x2="53.34" y2="33.02" width="0.508" layer="16"/>
-<wire x1="47.0662" y1="44.3738" x2="53.34" y2="38.1" width="0.508" layer="16"/>
-<wire x1="55.245" y1="17.145" x2="57.785" y2="19.685" width="0.508" layer="16"/>
+<wire x1="43.6372" y1="44.3738" x2="45.7962" y2="44.3738" width="0.508" layer="16"/>
+<wire x1="53.34" y1="36.83" x2="53.34" y2="33.02" width="0.508" layer="16"/>
+<wire x1="45.7962" y1="44.3738" x2="53.34" y2="36.83" width="0.508" layer="16"/>
+<wire x1="55.88" y1="17.78" x2="57.785" y2="19.685" width="0.508" layer="16"/>
 <wire x1="57.785" y1="19.685" x2="57.785" y2="26.67" width="0.508" layer="16"/>
-<wire x1="50.815125" y1="19.990125" x2="53.66025" y2="17.145" width="0.508" layer="16"/>
-<wire x1="53.66025" y1="17.145" x2="55.245" y2="17.145" width="0.508" layer="16"/>
+<wire x1="50.815125" y1="19.990125" x2="53.02525" y2="17.78" width="0.508" layer="16"/>
+<wire x1="53.02525" y1="17.78" x2="55.88" y2="17.78" width="0.508" layer="16"/>
 <wire x1="57.785" y1="26.67" x2="53.34" y2="31.115" width="0.508" layer="16"/>
 </signal>
@@
 <wire x1="40.005" y1="9.36625" x2="40.03881875" y2="9.21381875" width="0.5" layer="16"/>
 <wire x1="16.51" y1="19.52625" x2="16.383" y2="19.6088" width="0.5" layer="16"/>
-<wire x1="41.11625" y1="41.91" x2="41.11625" y2="44.29125" width="0.5" layer="16"/>
+<wire x1="41.11625" y1="40.79875" x2="41.11625" y2="44.29125" width="0.5" layer="16"/>
 <wire x1="41.11625" y1="44.29125" x2="41.0972" y2="44.3738" width="0.5" layer="16"/>
 <wire x1="11.27125" y1="31.90875" x2="11.2268" y2="32.004" width="0.5" layer="16"/>
@@
 <wire x1="46.355" y1="31.877" x2="46.228" y2="32.004" width="0.508" layer="16"/>
 <wire x1="46.228" y1="32.004" x2="46.228" y2="34.57575" width="0.508" layer="16"/>
-<wire x1="41.91" y1="40.005" x2="41.91" y2="41.275" width="0.508" layer="16"/>
-<wire x1="41.91" y1="41.275" x2="41.275" y2="41.91" width="0.508" layer="16"/>
-<wire x1="41.275" y1="41.91" x2="41.11625" y2="41.91" width="0.508" layer="16"/>
+<wire x1="46.355" y1="35.56" x2="41.11625" y2="40.79875" width="0.508" layer="16"/>
 <wire x1="41.0972" y1="44.3738" x2="39.9034" y2="43.18" width="0.508" layer="16"/>
 <wire x1="29.21" y1="52.07" x2="28.575" y2="51.435" width="0.508" layer="16"/>
@@
 <wire x1="9.144" y1="32.004" x2="8.255" y2="31.115" width="0.508" layer="16"/>
 <wire x1="8.255" y1="31.115" x2="8.255" y2="25.4" width="0.508" layer="16"/>
-<wire x1="41.91" y1="40.005" x2="46.355" y2="35.56" width="0.508" layer="16"/>
 <wire x1="46.355" y1="35.56" x2="46.355" y2="31.877" width="0.508" layer="16"/>
 </signal>

Commit message: modified IR-TX
Routing:
- net N$5: track 49.4 -> 48.9 mm
Changed lines of the file:
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@@
 <setting verticaltext="up"/>
 </settings>
-<grid distance="25" unitdist="mil" unit="mil" style="lines" multiple="1" display="no" altdistance="5" altunitdist="mil" altunit="mil"/>
+<grid distance="25" unitdist="mil" unit="mm" style="lines" multiple="1" display="no" altdistance="5" altunitdist="mil" altunit="mil"/>
 <layers>
 <layer number="1" name="Top" color="4" fill="1" visible="yes" active="yes"/>
@@
 <wire x1="41.43375" y1="27.46375" x2="41.43375" y2="36.83" width="0.508" layer="16"/>
 <wire x1="39.6875" y1="25.7175" x2="41.43375" y2="27.46375" width="0.508" layer="16"/>
-<wire x1="46.355" y1="19.685" x2="47.52815" y2="19.685" width="0.508" layer="16"/>
-<wire x1="47.52815" y1="19.685" x2="49.019075" y2="18.194075" width="0.508" layer="16"/>
-<wire x1="40.48125" y1="18.0975" x2="44.7675" y2="18.0975" width="0.508" layer="16"/>
-<wire x1="44.7675" y1="18.0975" x2="46.355" y2="19.685" width="0.508" layer="16"/>
+<wire x1="46.355" y1="19.05" x2="48.16315" y2="19.05" width="0.508" layer="16"/>
+<wire x1="48.16315" y1="19.05" x2="49.019075" y2="18.194075" width="0.508" layer="16"/>
+<wire x1="40.48125" y1="18.0975" x2="45.4025" y2="18.0975" width="0.508" layer="16"/>
+<wire x1="45.4025" y1="18.0975" x2="46.355" y2="19.05" width="0.508" layer="16"/>
 </signal>
 <signal name="N$6">
