File: PCB/MAIN/07/BOTTOM_BRD_v.1.0.3.sch (EAGLE design)
At the start: 66 parts, among them Q1 SS8050, Q2 SS8050, Q4 TIP122, SW1 CS12ANW03, U1 ESP32-WROOM-32D, U2 L293D, U3 AP2112K-3.3, U4 CE8301

Commit message: pcb v1.0.3 updates
Other:
- note added: "Swarmesh 2020 v1.0.3"
- note removed: "Swarmesh 2020 v1.0.2"
Changed lines of the file:
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@@
 other pins on IMU</text>
 <text x="135.255" y="60.96" size="1.778" layer="91">Note: Reset Button</text>
-<text x="229.87" y="-59.69" size="2.286" layer="94">Swarmesh 2020 v1.0.2</text>
+<text x="229.87" y="-59.69" size="2.286" layer="94">Swarmesh 2020 v1.0.3</text>
 <text x="176.53" y="-68.58" size="2.286" layer="94">NYU SHANGHAI
 SWARM ROBOTICS 2020

Commit message: pcb v1.0.3 updates
Parts:
- XR1, XR2, XR3, XR4, XR5: value TCRT1000 -> ST188
Changed lines of the file:
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@@
 <part name="GND29" library="supply1" deviceset="GND" device=""/>
 <part name="GND31" library="supply1" deviceset="GND" device=""/>
-<part name="XR1" library="ST188" deviceset="TCRT1000" device=""/>
-<part name="XR2" library="ST188" deviceset="TCRT1000" device=""/>
-<part name="XR3" library="ST188" deviceset="TCRT1000" device=""/>
-<part name="XR4" library="ST188" deviceset="TCRT1000" device=""/>
-<part name="XR5" library="ST188" deviceset="TCRT1000" device=""/>
+<part name="XR1" library="ST188" deviceset="TCRT1000" device="" value="ST188"/>
+<part name="XR2" library="ST188" deviceset="TCRT1000" device="" value="ST188"/>
+<part name="XR3" library="ST188" deviceset="TCRT1000" device="" value="ST188"/>
+<part name="XR4" library="ST188" deviceset="TCRT1000" device="" value="ST188"/>
+<part name="XR5" library="ST188" deviceset="TCRT1000" device="" value="ST188"/>
 <part name="Q4" library="TIP122" deviceset="TIP122" device="" value="TIP122"/>
 <part name="RB" library="rcl" library_urn="urn:adsk.eagle:library:334" deviceset="R-US_" device="M0805" package3d_urn="urn:adsk.eagle:package:23556/2" value="1k"/>
