File: PCB/MAIN/07/BOTTOM_BRD_v.1.0.3.brd (EAGLE design)
At the start: 99.1 x 85.8 mm, 66 parts, among them Q1 SS8050, Q2 SS8050, Q4 TIP122, SW1 CS12ANW03, U1 ESP32-WROOM-32D, U2 L293D, U3 AP2112K-3.3, U4 CE8301

Commit message: pcb v1.0.3 updates
Parts:
- moved R14 12.7 mm to (-41.9, 0.00), turned to 180 degrees
- moved R11 12.6 mm to (-29.2, -15.2)
- moved D1 11.7 mm to (11.4, 17.8), turned to 0 degrees
- moved R10 11.5 mm to (-31.8, -22.9), turned to 180 degrees
- moved R18 11.0 mm to (-31.8, 23.0), turned to 180 degrees
- moved R12 10.2 mm to (-38.1, -14.0), turned to 180 degrees
- moved R16 10.2 mm to (-38.1, 14.0), turned to 180 degrees
- moved L1 8.98 mm to (20.3, 10.2)
- moved C4 7.73 mm to (11.4, 11.4)
- moved R17 5.39 mm to (-31.8, 7.62)
- moved R4 5.08 mm to (21.6, -3.81)
- moved R5 5.08 mm to (26.7, -3.81)
- moved R13 4.02 mm to (-29.2, -12.7)
- moved C3 3.24 mm to (18.4, 15.2), turned to 0 degrees
- moved R20 1.80 mm to (31.8, -6.35)
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Routing:
- net +3V3: track 0.00 -> 248.1 mm, vias 0 -> 6
- net IR2: track 0.00 -> 160.9 mm, vias 0 -> 10
- net N$8: track 0.00 -> 139.0 mm, vias 0 -> 2
- net IO15: track 0.00 -> 138.8 mm, vias 0 -> 7
- net IO27: track 0.00 -> 136.8 mm, vias 0 -> 2
- net GND: track 338.2 -> 469.0 mm, vias 2 -> 7
- net N$9: track 0.00 -> 120.3 mm, vias 0 -> 6
- net EN: track 0.00 -> 105.5 mm, vias 0 -> 4
- net VCC: track 34.9 -> 136.1 mm, vias 0 -> 5
- net RXD: track 0.00 -> 100.7 mm, vias 0 -> 4
- net TOUCH1: track 0.00 -> 90.7 mm, vias 0 -> 3
- net IO32: track 0.00 -> 75.9 mm, vias 0 -> 2
- net +5V: track 165.1 -> 240.8 mm, vias 0 -> 1
- net TXD: track 0.00 -> 71.3 mm, vias 0 -> 3
- net IO5: track 0.00 -> 68.4 mm, vias 0 -> 3
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
Commit message: pcb v1.0.3 updates
Parts:
- XR1, XR2, XR3, XR4, XR5: value TCRT1000 -> ST188
- moved R14 13.3 mm to (-38.1, -12.7)
- moved R12 1.80 mm to (-36.8, -15.2)
- moved C1 1.80 mm to (22.9, 6.35)
- moved C6 1.80 mm to (17.8, 6.35)
- moved L1 1.27 mm to (20.3, 11.4)
- moved C3 0.90 mm to (17.8, 15.9)
Routing:
- net GND: track 469.0 -> 518.5 mm, vias 7 -> 6
- net N$10: track 5.07 -> 17.8 mm
- net +5V: track 240.8 -> 245.7 mm
- net IO39: track 25.2 -> 30.0 mm
- net N$9: track 120.3 -> 125.0 mm
- net IO34: track 53.2 -> 56.6 mm
- net IO0: track 59.3 -> 62.1 mm
- net VCC: track 136.1 -> 138.8 mm
- net EN: track 105.5 -> 107.6 mm
- net IO15: track 138.8 -> 140.5 mm
- net IO27: track 136.8 -> 135.2 mm
- net +3V3: track 248.1 -> 249.5 mm
- net E1A: track 58.0 -> 59.2 mm
- net IR2: track 160.9 -> 159.8 mm
- net N$8: track 139.0 -> 138.1 mm
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
Commit message: Update BOTTOM_BRD_v.1.0.3.brd
Routing:
- net E2A: track 63.4 -> 65.1 mm
- net M2B: track 61.4 -> 60.6 mm
- net GND: track 518.5 -> 519.1 mm
Other:
- board text added: "IR2"
- board text added: "SWARMESH 2020 2020/07/11 v1.0.3"
- board text removed: "M2 VCC C2 C1 GND M1"
- board text removed: "SWARMESH 2020 2020/07/10 v1.0.3"

Commit message: Update pcb v1.0.3
Parts:
- XR1, XR2, XR3, XR4, XR5: value ST188 -> TCRT1000
- moved C6 41.3 mm to (-22.9, 14.0), turned to 0 degrees
- moved C1 10.8 mm to (15.2, -1.27), turned to 0 degrees
- moved R4 5.08 mm to (26.7, -3.81)
- moved R5 5.08 mm to (21.6, -3.81)
- moved C2 5.08 mm to (15.2, 1.27), turned to 0 degrees
- moved U3 4.62 mm to (16.5, 5.71), turned to 270 degrees
- moved R19 2.54 mm to (-22.9, 16.5), turned to 0 degrees
- moved C9 1.27 mm to (20.3, -22.9)
- moved U4 0.25 mm to (21.6, 19.7)
- turned C5 to 0 degrees
Routing:
- net IO14: track 66.6 -> 150.0 mm, vias 3 -> 5
- net IR2: track 159.8 -> 77.2 mm, vias 10 -> 6
- net IO15: track 140.5 -> 63.5 mm, vias 7 -> 1
- net IO27: track 135.2 -> 59.9 mm
- net M2A: track 52.9 -> 103.2 mm, vias 2 -> 0
- net N$8: track 138.1 -> 177.6 mm, vias 2 -> 4
- net N$9: track 125.1 -> 89.1 mm, vias 6 -> 4
- net DTR: track 36.3 -> 71.7 mm, vias 1 -> 0
- net IO0: track 62.1 -> 29.7 mm, vias 0 -> 2
- net +5V: track 245.7 -> 277.9 mm, vias 1 -> 0
- net IO32: track 76.3 -> 103.6 mm, vias 2 -> 3
- net TOUCH1: track 91.1 -> 116.2 mm, vias 3 -> 5
- net +3V3: track 249.5 -> 274.5 mm, vias 6 -> 3
- net E1A: track 59.2 -> 37.5 mm, vias 2 -> 3
- net GND: track 519.1 -> 498.2 mm, vias 6 -> 4
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Other:
- board text added: "3V3 GND D0"
- board text added: "SWARMESH 2020 2020/07/12 v1.0.3"
- board text removed: "D0 GND 3V3"
- board text removed: "SWARMESH 2020 2020/07/11 v1.0.3"
