File: PCB/MAIN/07b/BOTTOM_BRD_v.1.0.5_c.sch (EAGLE design)
At the start: 66 parts, among them Q1 SS8050, Q2 SS8050, Q4 TIP122, SW1 CS12ANW03, U1 ESP32-WROOM-32D, U2 L293D, U3 AP2112K-3.3, U4 CE8301

Commit message: Update pcb v.1.0.3
Changed lines of the file:
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@@
 <wire x1="122.555" y1="78.74" x2="135.89" y2="78.74" width="0.1524" layer="91"/>
 <wire x1="122.555" y1="53.975" x2="122.555" y2="78.74" width="0.1524" layer="91"/>
+<junction x="122.555" y="78.74"/>
 </segment>
 </net>
