File: PCB/MAIN/08/BOTTOM_BRD_v.1.0.4.brd (EAGLE design)
At the start: 99.1 x 85.8 mm, 66 parts, among them Q1 SS8050, Q2 SS8050, Q4 TIP122, SW1 CS12ANW03, U1 ESP32-WROOM-32D, U2 L293D, U3 AP2112K-3.3, U4 CE8301

Commit message: PCB v1.0.4 Update
Parts:
- removed LED1\: LTE-302, LTE-302:LTE-302
- removed R20: 10, rcl:M0805
- T1: device Touch_Pad:SPRING-CONNECTOR -> Touch_Pad2:SPRING-CONNECTOR
- moved T1 2.80 mm to (-26.1, 34.2)
- moved T2 2.80 mm to (-26.1, -34.2)
- moved GPIO15 1.27 mm to (-17.8, 21.6)
- moved GPIO26 1.27 mm to (-15.2, 21.6)
- moved GPIO5 1.27 mm to (-20.3, 21.6)
- moved XR3 1.09 mm to (-43.0, 0.00)
- moved S1 1.00 mm to (17.8, 15.5)
- moved SW1 0.10 mm to (35.6, 17.9)
- flipped I2C to the top
Connections:
- removed net N$14: LED1\.A, R20.1
- net +5V: no longer R20.2
- net N$8: no longer LED1\.C
Routing:
- net N$8: track 177.6 -> 60.7 mm, vias 4 -> 1
- net DTR: track 71.7 -> 51.6 mm
- net GND: track 498.2 -> 482.4 mm, vias 4 -> 3
- net N$14: track 13.9 -> 0.00 mm
- net TOUCH1: track 116.2 -> 123.4 mm, vias 5 -> 6
- net +5V: track 277.9 -> 271.1 mm
- net +3V3: track 274.5 -> 281.0 mm, vias 3 -> 1
- net IO14: track 150.0 -> 154.3 mm
- net RTS: track 35.3 -> 32.2 mm, vias 4 -> 1
- net RXD: track 98.5 -> 95.5 mm
- net TOUCH2: track 44.1 -> 47.1 mm, vias 3 -> 4
- net VCC: track 121.8 -> 124.2 mm, vias 5 -> 3
- net EN: track 98.4 -> 100.0 mm
- net N$10: track 17.1 -> 18.7 mm
- net IO15: track 63.5 -> 62.2 mm
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Other:
- board text added: "SWARMESH 2020 2020/07/22 v1.0.4"
- board text removed: "SWARMESH 2020 2020/07/12 v1.0.3"
