File: PCB/MAIN/08/BOTTOM_BRD_v.1.0.4.sch (EAGLE design)
At the start: 66 parts, among them Q1 SS8050, Q2 SS8050, Q4 TIP122, SW1 CS12ANW03, U1 ESP32-WROOM-32D, U2 L293D, U3 AP2112K-3.3, U4 CE8301

Commit message: PCB v1.0.4 Update
Parts:
- removed LED1\: LTE-302, LTE-302:LTE-302
- removed R20: 10, rcl:R-US_M0805
- T1: device Touch_Pad:CONN_01SPRING-CONN -> Touch_Pad2:CONN_01SPRING-CONN
Connections:
- removed net N$14: LED1\.A, R20.1
- net +5V: no longer R20.2
- net N$8: no longer LED1\.C
Changed lines of the file:
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@@
 <part name="L1" library="SDR0604-100KL" deviceset="SDR0604-100KL" device="" value="47uH"/>
 <part name="GND21" library="supply1" deviceset="GND" device=""/>
-<part name="T1" library="Touch_Pad" deviceset="CONN_01" device="SPRING-CONN" package3d_urn="urn:adsk.eagle:package:38034/1"/>
+<part name="T1" library="Touch_Pad2" deviceset="CONN_01" device="SPRING-CONN" package3d_urn="urn:adsk.eagle:package:38034/1"/>
 <part name="T2" library="Touch_Pad" deviceset="CONN_01" device="SPRING-CONN" package3d_urn="urn:adsk.eagle:package:38034/1"/>
 <part name="U$2" library="No Connect NC" deviceset="NC" device=""/>
@@
 <part name="P+20" library="supply1" library_urn="urn:adsk.eagle:library:371" deviceset="+5V" device=""/>
 <part name="P+21" library="supply1" library_urn="urn:adsk.eagle:library:371" deviceset="+5V" device=""/>
-<part name="R20" library="rcl" library_urn="urn:adsk.eagle:library:334" deviceset="R-US_" device="M0805" package3d_urn="urn:adsk.eagle:package:23556/2" value="10"/>
-<part name="P+22" library="supply1" library_urn="urn:adsk.eagle:library:371" deviceset="+5V" device=""/>
-<part name="LED1\" library="LTE-302" deviceset="LTE-302" device=""/>
 <part name="+3V12" library="supply1" library_urn="urn:adsk.eagle:library:371" deviceset="+3V3" device=""/>
 <part name="+3V13" library="supply1" library_urn="urn:adsk.eagle:library:371" deviceset="+3V3" device=""/>
@@
 <attribute name="VALUE" x="218.7575" y="35.2425" size="1.778" layer="96" rot="MR0"/>
 </instance>
-<instance part="R20" gate="G$1" x="172.4025" y="34.6075" smashed="yes" rot="MR0">
-<attribute name="NAME" x="173.6725" y="36.1061" size="1.778" layer="95" rot="MR0"/>
-<attribute name="VALUE" x="177.4825" y="36.3855" size="1.27" layer="96" rot="MR0"/>
-</instance>
-<instance part="P+22" gate="1" x="164.7825" y="39.0525" smashed="yes" rot="MR0">
-<attribute name="VALUE" x="166.37" y="40.005" size="1.778" layer="96" rot="MR0"/>
-</instance>
-<instance part="LED1\" gate="G$1" x="182.88" y="34.6075" smashed="yes" rot="R90">
-<attribute name="VALUE" x="180.723940625" y="30.92198125" size="1.27" layer="96"/>
-<attribute name="NAME" x="181.35931875" y="38.03555" size="1.778" layer="95"/>
-</instance>
 <instance part="+3V12" gate="G$1" x="-60.6425" y="6.985" smashed="yes">
 <attribute name="VALUE" x="-58.1025" y="9.525" size="1.778" layer="96" rot="R180"/>
@@
 <wire x1="217.17" y1="31.75" x2="217.17" y2="30.48" width="0.1524" layer="91"/>
 <pinref part="P+21" gate="1" pin="+5V"/>
-</segment>
-<segment>
-<pinref part="R20" gate="G$1" pin="2"/>
-<pinref part="P+22" gate="1" pin="+5V"/>
-<wire x1="167.3225" y1="34.6075" x2="164.7825" y2="34.6075" width="0.1524" layer="91"/>
-<wire x1="164.7825" y1="34.6075" x2="164.7825" y2="36.5125" width="0.1524" layer="91"/>
 </segment>
 </net>
@@
 <junction x="203.2" y="58.42"/>
 <junction x="203.2" y="25.4"/>
-<wire x1="195.58" y1="25.4" x2="195.58" y2="34.6075" width="0.1524" layer="91"/>
-<wire x1="195.58" y1="34.6075" x2="187.96" y2="34.6075" width="0.1524" layer="91"/>
-<junction x="195.58" y="25.4"/>
-<pinref part="LED1\" gate="G$1" pin="C"/>
 </segment>
 </net>
@@
 </segment>
 </net>
-<net name="N$14" class="0">
-<segment>
-<pinref part="R20" gate="G$1" pin="1"/>
-<wire x1="177.4825" y1="34.6075" x2="180.34" y2="34.6075" width="0.1524" layer="91"/>
-<pinref part="LED1\" gate="G$1" pin="A"/>
-</segment>
-</net>
